File: denton-rain-maker.kicad_pcb (KiCad board)
At the start: 2 copper layers, 63 parts, among them J1 Live(AC2), J2 Neutral(AC1), J3 SEED C3, Q1 BT136S-800E, Q2 BT136S-800E, Q3 BT136S-800E, Q4 BT136S-800E, U1 MOC3063M, U2 MOC3063M, U3 MOC3063M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

Commit message: starting on layout
Parts:
- removed D2, D5, D7: LED, LED_SMD:LED_1206_3216Metric_Pad1.42x1.75mm_HandSolder
- removed D3, D4, D6: 1N4148W, Diode_SMD:D_SOD-123
- removed J2: Neutral(AC1), Connector_PinSocket_1.27mm:PinSocket_1x01_P1.27mm_Vertical
- removed Q1, Q2, Q3: BT136S-800E, Package_TO_SOT_SMD:TO-252-3_TabPin2
- removed R1, R16, R17, R18, R19, R20, R9: 10k, Resistor_SMD:R_1206_3216Metric_Pad1.30x1.75mm_HandSolder
- removed R11, R12, R2, R22, R23, R3: 220, Resistor_SMD:R_1206_3216Metric_Pad1.30x1.75mm_HandSolder
- removed U1, U2, U3: MOC3063M, Package_DIP:DIP-6_W7.62mm
- added D10: LED, LED_THT:LED_D3.0mm, F.Cu at (158.5, 40.0)
- added D11: LED, LED_THT:LED_D3.0mm, F.Cu at (123.0, 82.0)
- added D12: 1N4148W, Diode_SMD:D_SOD-123, F.Cu at (107.9, 165.0)
- added D13: LED, LED_THT:LED_D3.0mm, F.Cu at (110.5, 180.0)
- added D14: 1N4148W, Diode_SMD:D_SOD-123, F.Cu at (83.7, 165.5)
- added D15: LED, LED_THT:LED_D3.0mm, F.Cu at (91.5, 187.0)
- added D16: 1N4148W, Diode_SMD:D_SOD-123, F.Cu at (60.8, 174.5)
- added D17: LED, LED_THT:LED_D3.0mm, F.Cu at (56.0, 186.0)
- added Q5: BT136S-800E, Package_TO_SOT_SMD:TO-252-3_TabPin2, F.Cu at (110.4, 149.5)
- added Q6: BT136S-800E, Package_TO_SOT_SMD:TO-252-3_TabPin2, F.Cu at (89.0, 153.3)
- added Q7: BT136S-800E, Package_TO_SOT_SMD:TO-252-3_TabPin2, F.Cu at (65.3, 156.3)
- added R25: 10k, Resistor_SMD:R_1206_3216Metric_Pad1.30x1.75mm_HandSolder, F.Cu at (116.5, 160.0)
- added R38: 220, Resistor_SMD:R_1206_3216Metric_Pad1.30x1.75mm_HandSolder, F.Cu at (93.5, 142.0)
- added R39: 100, Resistor_SMD:R_1206_3216Metric_Pad1.30x1.75mm_HandSolder, F.Cu at (69.5, 186.0)
- added R40: 220, Resistor_SMD:R_1206_3216Metric_Pad1.30x1.75mm_HandSolder, F.Cu at (58.5, 143.0)
- added R41: 10k, Resistor_SMD:R_1206_3216Metric_Pad1.30x1.75mm_HandSolder, F.Cu at (48.5, 146.0)
- added R42: 220, Resistor_SMD:R_1206_3216Metric_Pad1.30x1.75mm_HandSolder, F.Cu at (62.5, 115.0)
- added R43: 220, Resistor_SMD:R_1206_3216Metric_Pad1.30x1.75mm_HandSolder, F.Cu at (67.5, 143.0)
- added R44: 100, Resistor_SMD:R_1206_3216Metric_Pad1.30x1.75mm_HandSolder, F.Cu at (50.5, 168.0)
- added S1: RDS7-8S-1065-73-D-67, Downloads:SW_RDS7-8S-1065-73-D-67, F.Cu at (118.0, 59.7)
- added U6: MOC3063M, Package_DIP:DIP-6_W7.62mm, F.Cu at (104.2, 127.2)
- added U7: MOC3063M, Package_DIP:DIP-6_W7.62mm, F.Cu at (84.9, 127.6)
- added U8: MOC3063M, Package_DIP:DIP-6_W7.62mm, F.Cu at (61.2, 127.5)
- D9: footprint LED_SMD:LED_1206_3216Metric_Pad1.42x1.75mm_HandSolder -> LED_THT:LED_D3.0mm
- J1: value Live(AC2) -> Conn_01x06; footprint Connector_PinSocket_1.27mm:PinSocket_1x01_P1.27mm_Vertical -> TerminalBlock_Phoenix:TerminalBlock_Phoenix_MPT-0,5-6-2.54_1x06_P2.54mm_Horizontal
- R28, R29, R30, R31, R36: value 10k -> 220
- R34: value 100 -> 220
- R35: value 100 -> 10k
- R5: value 30k -> 220
- moved C7 129.4 mm to (71.6, 175.0)
- moved C5 111.6 mm to (94.3, 168.0)
- moved R35 109.4 mm to (68.5, 168.0)
- moved C6 97.6 mm to (115.4, 172.0)
- moved R6 93.1 mm to (220.4, 75.0)
- moved R33 84.7 mm to (103.5, 158.0)
- moved R34 83.1 mm to (83.5, 142.0)
- moved U5 82.6 mm to (211.9, 61.2)
- moved D1 81.4 mm to (233.5, 61.5)
- moved R8 81.4 mm to (189.4, 47.0)
- moved R7 72.0 mm to (178.4, 46.0)
- moved R37 71.2 mm to (165.4, 30.0)
- moved C12 70.0 mm to (174.7, 62.2)
- moved J1 69.4 mm to (160.0, 173.5)
- moved R36 64.9 mm to (85.5, 115.0)
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Connections:
- C4 pad 2: Net-(J2-Pin_1) -> Net-(D8-K)
- C5 pad 2: Net-(J2-Pin_1) -> Net-(D12-K)
- C6 pad 2: Net-(J2-Pin_1) -> Net-(D14-K)
- C7 pad 2: Net-(J2-Pin_1) -> Net-(D16-K)
- D1 pad 1: Net-(D3-K) -> /LINE_IN
- D1 pad 2: Net-(J2-Pin_1) -> NEUT
- D8 pad 1: Net-(D3-K) -> Net-(D8-K)
- D8 pad 2: Net-(D8-A) -> NEUT
- D9 pad 1: Net-(D8-A) -> NEUT
- J1 pad 1: Net-(D3-K) -> Net-(D16-K)
- J3 pad 3: unconnected-(J3-Pin_7-Pad3) -> Net-(J3-Pin_7-Pad3)
- J3 pad 4: unconnected-(J3-Pin_6-Pad4) -> Net-(J3-Pin_6-Pad4)
- J3 pad 5: unconnected-(J3-Pin_5-Pad5) -> Net-(J3-Pin_5-Pad5)
- Q4 pad 1: Net-(J2-Pin_1) -> Net-(D8-K)
- Q4 pad 2: Net-(D3-K) -> /LINE_IN
- R13 pad 1: Net-(J3-Pin_8) -> Net-(J3-Pin_3-Pad3.3V)
- R13 pad 2: Net-(J3-Pin_8) -> Net-(J3-Pin_7-Pad3)
- R14 pad 1: Net-(J3-Pin_8) -> Net-(J3-Pin_3-Pad3.3V)
- R15 pad 1: Net-(J3-Pin_8) -> Net-(J3-Pin_3-Pad3.3V)
- R15 pad 2: Net-(J3-Pin_8) -> Net-(J3-Pin_6-Pad4)
- R24 pad 2: Net-(J2-Pin_1) -> Net-(D8-K)
- R27 pad 2: Net-(D3-K) -> /LINE_IN
- R28 pad 1: Net-(Q4-G) -> Net-(R28-Pad1)
- R28 pad 2: Net-(J2-Pin_1) -> Net-(Q4-G)
- R29 pad 2: Net-(J2-Pin_1) -> Net-(Q5-G)
- R30 pad 2: Net-(J2-Pin_1) -> Net-(J3-Pin_7-Pad20)
- R31 pad 2: Net-(J2-Pin_1) -> /LINE_IN
- R32 pad 1: Net-(D3-K) -> /LINE_IN
- R33 pad 1: Net-(D3-K) -> /LINE_IN
- R34 pad 1: Net-(D3-K) -> Net-(R34-Pad1)
- R34 pad 2: Net-(C6-Pad1) -> Net-(Q6-G)
- R35 pad 1: Net-(D3-K) -> Net-(D15-A)
- R35 pad 2: Net-(C7-Pad1) -> Net-(D14-K)
- R36 pad 1: GND -> Net-(R36-Pad1)
- R36 pad 2: Net-(J3-Pin_8) -> Net-(J3-Pin_2-Pad21)
- R5 pad 1: Net-(J3-Pin_3-Pad3.3V) -> Net-(D11-A)
- R5 pad 2: Net-(J3-Pin_8) -> Net-(J3-Pin_5-Pad5)
- U4 pad 4: Net-(Q4-G) -> Net-(R28-Pad1)
Other:
- board outline added: 100 x 100 mm

Commit message: layout continues
Parts:
- added L1: 47uH, Inductor_SMD:L_Bourns_SRN6045TA, F.Cu at (197.5, 58.3)
- moved C12 50.4 mm to (221.0, 82.0)
- moved R7 34.4 mm to (206.0, 66.5), turned to -90 degrees
- moved R26 33.5 mm to (163.0, 111.5), turned to 90 degrees
- moved C1 29.3 mm to (219.4, 75.0)
- moved D1 28.5 mm to (213.7, 82.1), turned to 90 degrees
- moved R8 23.2 mm to (202.0, 66.5), turned to -90 degrees
- moved J1 16.1 mm to (164.3, 158.0)
- moved C3 15.6 mm to (177.0, 59.0), turned to -90 degrees
- moved C2 14.0 mm to (210.4, 54.0)
- moved C11 13.8 mm to (213.4, 75.0), turned to 180 degrees
- moved R6 9.56 mm to (219.0, 65.5), turned to -90 degrees
- moved D9 9.43 mm to (164.5, 146.0)
- moved U4 8.06 mm to (163.0, 116.4)
- moved R24 5.10 mm to (168.4, 140.0)
- moved R28 4.24 mm to (155.0, 128.6)
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
Commit message: gotta stop
Parts:
- added C8: 100nF, Capacitor_SMD:C_1206_3216Metric_Pad1.33x1.80mm_HandSolder, F.Cu at (169.0, 60.6)
- added C9: 10uF, Capacitor_SMD:C_1206_3216Metric_Pad1.33x1.80mm_HandSolder, F.Cu at (174.0, 60.6)
- moved R37 36.7 mm to (169.0, 66.5), turned to 90 degrees
- moved D10 30.0 mm to (175.0, 65.0), turned to -90 degrees
- moved R15 26.3 mm to (140.6, 51.9)
- moved S1 24.2 mm to (142.0, 62.0), turned to 180 degrees
- moved R7 20.6 mm to (222.0, 53.5)
- moved R8 19.8 mm to (217.0, 53.5)
- moved L1 17.5 mm to (210.9, 47.0)
- moved D11 16.3 mm to (135.0, 71.0), turned to -90 degrees
- moved R14 13.6 mm to (135.4, 66.9)
- moved R13 7.87 mm to (134.4, 52.0)
- moved C3 5.00 mm to (182.0, 59.0)
- moved R5 4.03 mm to (141.4, 72.0), turned to 90 degrees
- moved R6 3.16 mm to (218.0, 62.5), turned to 90 degrees
- moved C2 1.00 mm to (210.4, 55.0), turned to 180 degrees
Connections:
- R13 pad 2: Net-(J3-Pin_7-Pad3) -> Net-(J3-Pin_6-Pad4)
- R14 pad 2: Net-(J3-Pin_8) -> Net-(J3-Pin_7-Pad3)
- R15 pad 2: Net-(J3-Pin_6-Pad4) -> Net-(J3-Pin_8)
- S1 pad 1: Net-(J3-Pin_8) -> Net-(J3-Pin_7-Pad3)
- S1 pad 2: Net-(J3-Pin_7-Pad3) -> Net-(J3-Pin_6-Pad4)
- S1 pad 4: Net-(J3-Pin_6-Pad4) -> Net-(J3-Pin_8)

Commit message: remember to change the buck converter
Parts:
- C8, C9, R13, R14, R15, R37: moved to B.Cu
- U5: footprint Package_SO:HSOP-8-1EP_3.9x4.9mm_P1.27mm_EP2.41x3.1mm_ThermalVias -> Package_SO:Texas_R-PDSO-G8_EP2.95x4.9mm_Mask2.4x3.1mm
- moved R39 120.8 mm to (149.5, 95.4), turned to -90 degrees
- moved R44 110.2 mm to (133.5, 95.4), turned to -90 degrees
- moved D17 101.2 mm to (126.5, 113.4), turned to 180 degrees
- moved R35 100.5 mm to (149.9, 109.0)
- moved C5 97.2 mm to (165.2, 101.4), turned to -90 degrees
- moved C7 96.2 mm to (133.5, 101.4), turned to -90 degrees
- moved D16 94.1 mm to (132.3, 113.4), turned to 180 degrees
- moved R41 93.1 mm to (133.9, 108.9)
- moved D15 89.9 mm to (143.0, 113.4), turned to 180 degrees
- moved R33 87.9 mm to (165.2, 95.4), turned to -90 degrees
- moved U8 83.3 mm to (131.5, 82.9), turned to -90 degrees
- moved D14 83.0 mm to (148.3, 113.4), turned to 180 degrees
- moved R40 82.9 mm to (126.5, 95.4), turned to -90 degrees
- moved D13 81.8 mm to (158.2, 113.5), turned to 180 degrees
- moved Q7 79.8 mm to (127.2, 105.9), turned to -90 degrees
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Connections:
- C3 pad 1: Net-(J3-Pin_1) -> Net-(D10-A)
- C8 pad 1: Net-(J3-Pin_1) -> Net-(D10-A)
- C9 pad 1: Net-(J3-Pin_1) -> Net-(D10-A)
- D10 pad 1: GND -> Net-(D10-K)
- J3 pad 5V: Net-(J3-Pin_1) -> Net-(D10-A)
- L1 pad 2: Net-(J3-Pin_1) -> Net-(D10-A)
- R28 pad 1: Net-(R28-Pad1) -> Net-(Q4-G)
- R28 pad 2: Net-(Q4-G) -> Net-(D8-K)
- R29 pad 1: Net-(R29-Pad1) -> Net-(Q5-G)
- R29 pad 2: Net-(Q5-G) -> Net-(D12-K)
- R34 pad 1: Net-(R34-Pad1) -> Net-(Q6-G)
- R34 pad 2: Net-(Q6-G) -> Net-(D14-K)
- R37 pad 1: Net-(D10-A) -> GND
- R37 pad 2: Net-(J3-Pin_1) -> Net-(D10-K)
- R40 pad 1: Net-(R40-Pad1) -> Net-(Q7-G)
- R40 pad 2: Net-(Q7-G) -> Net-(D16-K)
- R8 pad 1: Net-(J3-Pin_1) -> Net-(D10-A)
- U4 pad 4: Net-(R28-Pad1) -> Net-(Q4-G)
- U6 pad 4: Net-(R29-Pad1) -> Net-(Q5-G)
- U7 pad 4: Net-(R34-Pad1) -> Net-(Q6-G)
- U8 pad 4: Net-(R40-Pad1) -> Net-(Q7-G)
Routing:
- net /LINE_IN: track 0.00 -> 81.4 mm, vias 0 -> 8
- net Net-(D16-K): track 0.00 -> 72.2 mm, vias 0 -> 1
- net NEUT: track 0.00 -> 69.6 mm
- net Net-(D14-K): track 0.00 -> 54.9 mm, vias 0 -> 1
- net Net-(D12-K): track 0.00 -> 37.8 mm, vias 0 -> 1
- net Net-(J3-Pin_6-Pad4): track 0.00 -> 36.1 mm
- net Net-(D10-A): track 0.00 -> 35.0 mm
- net Net-(J3-Pin_3-Pad7): track 0.00 -> 22.1 mm
- net Net-(D8-K): track 0.00 -> 19.7 mm, vias 0 -> 1
- net Net-(J3-Pin_3-Pad3.3V): track 0.00 -> 18.7 mm, vias 0 -> 1
- net Net-(J3-Pin_6-Pad8): track 0.00 -> 15.6 mm
- net Net-(J3-Pin_8): track 0.00 -> 14.7 mm
- net Net-(J3-Pin_7-Pad3): track 0.00 -> 13.7 mm
- net Net-(D1-+): track 0.00 -> 13.2 mm
- net Net-(Q4-G): track 0.00 -> 11.3 mm
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Other:
- board size 100 x 100 mm -> 75 x 75 mm
- board text added: "0.)Program 1.)Off 2.)Auto 3.)Test 1 4.)Test 2 5.)Test 3 6.)Test 4 7.)Test 1-4 seq."

Commit message: added LDO,MOV
Parts:
- removed R6: 100k, Resistor_SMD:R_1206_3216Metric_Pad1.30x1.75mm_HandSolder
- removed U5: LM5164DDA, Package_SO:Texas_R-PDSO-G8_EP2.95x4.9mm_Mask2.4x3.1mm
- added C10: 22uF, Capacitor_SMD:C_1206_3216Metric_Pad1.33x1.80mm_HandSolder, F.Cu at (183.5, 61.6)
- added C13: 0.1uF, Capacitor_SMD:C_1206_3216Metric_Pad1.33x1.80mm_HandSolder, F.Cu at (168.0, 65.6)
- added F1: Fuse, Fuse:Fuseholder_Blade_Mini_Keystone_3568, F.Cu at (189.1, 116.4)
- added J2: MOV, Capacitor_THT:C_Disc_D7.5mm_W5.0mm_P7.50mm, F.Cu at (193.5, 100.0)
- added R9: 250k, Resistor_SMD:R_1206_3216Metric_Pad1.30x1.75mm_HandSolder, F.Cu at (194.0, 66.5)
- added U1: LMR38020FSDDAR, footprints:DDA0008E-IPC_C, F.Cu at (190.5, 72.5)
- added U2: TLV1117-33, Package_TO_SOT_SMD:SOT-223-3_TabPin2, F.Cu at (177.0, 60.1)
- C1, C11: moved to B.Cu
- C3: value 47uF -> 22uF; footprint Capacitor_THT:CP_Radial_D6.3mm_P2.50mm -> Capacitor_SMD:C_1206_3216Metric_Pad1.33x1.80mm_HandSolder
- C8: value 100nF -> 10uF; moved to F.Cu
- C9: value 10uF -> 1uF; moved to F.Cu
- R37: moved to F.Cu
- R7: value 10k -> 24.9k
- R8: value 31.6k -> 100k
- moved J1 31.6 mm to (161.8, 122.5), turned to 0 degrees
- moved R7 11.2 mm to (190.0, 66.5), turned to 90 degrees
- moved C9 10.5 mm to (187.5, 61.6), turned to 90 degrees
- moved D10 9.55 mm to (171.5, 79.0)
- moved C3 7.59 mm to (176.9, 67.5), turned to 180 degrees
- moved C11 6.52 mm to (190.9, 80.5)
- moved R8 5.83 mm to (184.4, 68.5)
- moved C2 5.44 mm to (184.0, 74.5)
- moved R37 5.32 mm to (171.5, 72.0)
- moved L1 5.02 mm to (178.5, 73.6)
- moved C12 4.30 mm to (192.5, 83.5)
- moved C1 4.27 mm to (190.9, 77.5), turned to 180 degrees
- moved C8 3.54 mm to (171.5, 65.6)
Connections:
- C3 pad 1: Net-(D10-A) -> Net-(U2-VI)
- C8 pad 1: Net-(D10-A) -> Net-(U2-VO)
- C9 pad 1: Net-(D10-A) -> Net-(U2-VI)
- D10 pad 1: Net-(D10-K) -> GND
- J3 pad 3.3V: Net-(J3-Pin_3-Pad3.3V) -> Net-(U2-VO)
- J3 pad 5V: Net-(D10-A) -> unconnected-(J3-Pin_1-Pad5V)
- J3 pad GND: GND -> unconnected-(J3-Pin_2-PadGND)
- L1 pad 2: Net-(D10-A) -> Net-(U2-VI)
- R13 pad 1: Net-(J3-Pin_3-Pad3.3V) -> Net-(U2-VO)
- R14 pad 1: Net-(J3-Pin_3-Pad3.3V) -> Net-(U2-VO)
- R15 pad 1: Net-(J3-Pin_3-Pad3.3V) -> Net-(U2-VO)
- R37 pad 1: GND -> Net-(D10-A)
- R37 pad 2: Net-(D10-K) -> Net-(U2-VI)
- R8 pad 1: Net-(D10-A) -> Net-(U2-VI)
Routing:
- net Net-(D10-A): track 35.0 -> 0.00 mm
- net Net-(J3-Pin_3-Pad3.3V): track 18.7 -> 0.00 mm, vias 1 -> 0
- net Net-(J3-Pin_6-Pad8): track 15.6 -> 0.00 mm
- net Net-(U2-VO): track 0.00 -> 14.2 mm, vias 0 -> 1
- net /LINE_IN: track 81.4 -> 67.8 mm
- net Net-(D1-+): track 13.2 -> 0.00 mm
- net Net-(U1-FB): track 11.0 -> 0.00 mm
- net NEUT: track 69.6 -> 59.4 mm
- net Net-(U1-SW): track 6.01 -> 0.00 mm
- net Net-(U5-RON): track 5.45 -> 0.00 mm
- net Net-(D10-K): track 5.24 -> 0.00 mm
- net Net-(D8-K): track 19.7 -> 17.5 mm, vias 1 -> 0

Commit message: new pwr supply
Parts:
- removed C10, C3: 22uF, Capacitor_SMD:C_1206_3216Metric_Pad1.33x1.80mm_HandSolder
- removed C2: 2.2nF, Capacitor_SMD:C_1206_3216Metric_Pad1.33x1.80mm_HandSolder
- removed L1: 47uH, Inductor_SMD:L_Bourns_SRN6045TA
- removed R7: 24.9k, Resistor_SMD:R_1206_3216Metric_Pad1.30x1.75mm_HandSolder
- removed R8: 100k, Resistor_SMD:R_1206_3216Metric_Pad1.30x1.75mm_HandSolder
- removed R9: 250k, Resistor_SMD:R_1206_3216Metric_Pad1.30x1.75mm_HandSolder
- added C14: 220uF, Capacitor_THT:CP_Radial_D10.0mm_P5.00mm, F.Cu at (161.7, 74.3)
- added D2: D_Schottky_Small, Diode_SMD:D_MicroSMP_LargeCathode, F.Cu at (169.9, 59.3)
- added L2: NRS6028T330MMGJ, inductor:IND_TAIYO_NRS6028_TAY, F.Cu at (164.9, 65.6)
- C1, C11: moved to F.Cu
- U1: value LMR38020FSDDAR -> LM2596S-5; footprint footprints:DDA0008E-IPC_C -> Package_TO_SOT_SMD:TO-263-5_TabPin3
- moved J1 38.7 mm to (123.3, 119.9)
- moved F1 37.3 mm to (151.8, 117.6), turned to 0 degrees
- moved J2 26.5 mm to (175.4, 119.3)
- moved D10 24.8 mm to (171.5, 54.2)
- moved C9 22.8 mm to (164.8, 58.9)
- moved R37 20.3 mm to (164.7, 52.9), turned to -90 degrees
- moved D1 19.7 mm to (181.7, 109.8)
- moved U2 19.7 mm to (158.1, 54.7)
- moved C8 15.9 mm to (155.6, 64.7)
- moved C1 14.7 mm to (176.3, 76.7), turned to 0 degrees
- moved C11 14.5 mm to (176.5, 80.4), turned to 0 degrees
- moved D11 14.2 mm to (129.5, 71.5)
- moved R5 14.2 mm to (128.5, 67.5)
- moved J3 13.5 mm to (142.9, 63.7)
- moved R13 13.5 mm to (140.8, 66.4)
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Connections:
- C9 pad 1: Net-(U2-VI) -> Net-(U1-FB)
- R37 pad 2: Net-(U2-VI) -> Net-(U1-FB)
- U1 pad 1: GND -> Net-(D1-+)
- U1 pad 2: Net-(D1-+) -> Net-(D2-K)
- U1 pad 3: Net-(D1-+) -> GND
- U1 pad 4: Net-(U1-RT_SYNC) -> Net-(U1-FB)
- U1 pad 5: Net-(U1-FB) -> GND
- U2 pad 3: Net-(U2-VI) -> Net-(U1-FB)
Routing:
- net Net-(D16-K): track 72.2 -> 18.3 mm
- net Net-(D14-K): track 54.9 -> 19.5 mm
- net Net-(J3-Pin_6-Pad4): track 36.1 -> 3.54 mm
- net Net-(J3-Pin_3-Pad7): track 22.1 -> 0.10 mm
- net Net-(D12-K): track 37.8 -> 20.4 mm
- net Net-(J3-Pin_8): track 14.7 -> 5.87 mm
- net Net-(J3-Pin_7-Pad3): track 13.7 -> 6.30 mm
- net Net-(J3-Pin_5-Pad5): track 6.20 -> 0.00 mm
- net Net-(J3-Pin_7-Pad20): track 6.08 -> 0.00 mm
- net Net-(J3-Pin_2-Pad21): track 5.80 -> 1.39 mm
- net Net-(R36-Pad1): track 4.08 -> 0.00 mm
- net Net-(R42-Pad1): track 5.29 -> 1.91 mm
- net Net-(R30-Pad1): track 4.14 -> 1.19 mm
Other:
- outline, holes or cut-outs redrawn
- board text added: "1 2 3 4 AC1 AC2"
- board text added: "B. LED"
- board text added: "G. LED"
- board text added: "R. LED"
